File: PowerStripper.kicad_pcb (KiCad board)
At the start: 2 copper layers, 33 x 25.4 mm, 5 parts, among them J1 0548190519, J2 UE27AC54100

Commit message: Worked on reorganizing in pcbnew
Parts:
- moved S1 16.3 mm to (119.6, 117.1), turned to 0 degrees
- moved R1 12.8 mm to (122.9, 93.7), turned to 180 degrees
- moved J2 11.7 mm to (108.2, 105.7)
- moved D1 5.64 mm to (130.0, 94.7)
- moved J1 4.68 mm to (130.3, 105.7)
Routing:
- net Net-(J2-Pad1): track 19.6 -> 48.8 mm
- net D-: track 17.7 -> 43.7 mm
- net D+: track 11.7 -> 25.1 mm
- net Net-(J1-Pad1): track 7.64 -> 19.6 mm
- removed copper zone on B.Cu, net GND
Other:
- board size 33 x 25.4 mm -> 57.9 x 31 mm
- net class USB added: clearance 0.2, trace_width 1.645046, via_dia 0.8, via_drill 0.4

Commit message: made changes to pcb
Parts:
- moved D1 16.0 mm to (114.0, 94.0)
- moved R1 15.2 mm to (107.7, 94.0)
- moved S1 5.40 mm to (116.1, 113.0)
- moved J1 5.08 mm to (125.2, 105.7)
Connections:
- J2 pad 1: Net-(J2-Pad1) -> GND
- R1 pad 2: Net-(J2-Pad1) -> GND
- S1 pad 1: Net-(J2-Pad1) -> GND
Routing:
- net Net-(J2-Pad1): track 48.8 -> 0.00 mm
- net D+: track 25.1 -> 52.2 mm
- net D-: track 43.7 -> 57.7 mm
- net Net-(J1-Pad1): track 19.6 -> 9.91 mm
- net Net-(D1-Pad1): track 4.99 -> 3.81 mm
- added copper zone on B.Cu, net GND
Other:
- net class USB: trace_width 1.645046 -> 3.4

Commit message: changed board size
Other:
- board size 57.9 x 31 mm -> 37.3 x 31 mm
Changed lines of the file:
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@@
   )
   (layers
-    (0 F.Cu signal)
+    (0 F.Cu signal hide)
     (31 B.Cu signal hide)
     (32 B.Adhes user)
@@
       (effects (font (size 1 1) (thickness 0.15)))
     )
-    (fp_text value UE27AC54100 (at 0 12 90) (layer F.Fab)
+    (fp_text value UE27AC54100 (at 9.652 3.556) (layer F.Fab)
       (effects (font (size 1 1) (thickness 0.15)))
     )
@@
     (effects (font (size 1 1) (thickness 0.15)))
   )
-  (gr_line (start 97.536 90.932) (end 155.448 90.932) (layer Edge.Cuts) (width 0.05))
+  (gr_line (start 97.536 90.932) (end 134.874 90.932) (layer Edge.Cuts) (width 0.05))
   (gr_line (start 97.536 121.92) (end 97.536 90.932) (layer Edge.Cuts) (width 0.05))
-  (gr_line (start 155.448 121.92) (end 97.536 121.92) (layer Edge.Cuts) (width 0.05))
-  (gr_line (start 155.448 90.932) (end 155.448 121.92) (layer Edge.Cuts) (width 0.05))
+  (gr_line (start 134.874 121.92) (end 97.536 121.92) (layer Edge.Cuts) (width 0.05))
+  (gr_line (start 134.874 90.932) (end 134.874 121.92) (layer Edge.Cuts) (width 0.05))
   (segment (start 110.998 102.08) (end 110.914 102.164) (width 0.25) (layer F.Cu) (net 1))
   (segment (start 110.858 102.108) (end 110.914 102.164) (width 0.25) (layer B.Cu) (net 1))

Commit message: made more changes to pcb
Parts:
- moved D1 0.25 mm to (114.0, 94.2)
- moved R1 0.25 mm to (107.7, 94.2)
Connections:
- J2 pad 1: GND -> Net-(J2-Pad1)
- R1 pad 2: GND -> Net-(J2-Pad1)
- S1 pad 1: GND -> Net-(J2-Pad1)
Routing:
- net Net-(J2-Pad1): track 0.00 -> 28.5 mm
- net D-: track 57.7 -> 55.5 mm
Other:
- net class Default: clearance 0.2 -> 0.1524
- net class USB: clearance 0.2 -> 0.1524
- rule trace_clearance: 0.2 -> 0.1524
- rule trace_min: 0.2 -> 0.152
Changed lines of the file:
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@@
     (thickness 1.6)
     (drawings 5)
-    (tracks 31)
+    (tracks 35)
     (zones 0)
     (modules 5)
-    (nets 8)
+    (nets 9)
   )
   (page A4)
@@
   )
   (layers
-    (0 F.Cu signal hide)
+    (0 F.Cu signal)
     (31 B.Cu signal hide)
     (32 B.Adhes user)
@@
   (setup
     (last_trace_width 0.25)
-    (trace_clearance 0.2)
+    (trace_clearance 0.1524)
     (zone_clearance 0.508)
     (zone_45_only no)
-    (trace_min 0.2)
+    (trace_min 0.152)
     (via_size 0.8)
     (via_drill 0.4)
@@
     (mod_text_size 1 1)
     (mod_text_width 0.15)
-    (pad_size 1.524 1.524)
-    (pad_drill 0.762)
+    (pad_size 1.65 1.1)
+    (pad_drill 0.7)
     (pad_to_mask_clearance 0)
     (aux_axis_origin 163.83 104.14)
@@
   (net 6 "Net-(J1-Pad4)")
   (net 7 "Net-(S1-Pad3)")
+  (net 8 "Net-(J2-Pad1)")
   (net_class Default "This is the default net class."
-    (clearance 0.2)
+    (clearance 0.1524)
     (trace_width 0.25)
     (via_dia 0.8)
@@
     (add_net "Net-(J1-Pad1)")
     (add_net "Net-(J1-Pad4)")
+    (add_net "Net-(J2-Pad1)")
     (add_net "Net-(S1-Pad3)")
   )
   (net_class USB ""
-    (clearance 0.2)
+    (clearance 0.1524)
     (trace_width 3.4)
     (via_dia 0.8)
@@
   )
   (module digikey-footprints:LED_3mm_Radial (layer F.Cu)
-    (at 114.046 93.98)
+    (at 114.046 94.234)
     (descr http://optoelectronics.liteon.com/upload/download/DS20-2000-343/1CHKxKNN.pdf)
     (fp_text reference D1 (at 2.54 0) (layer F.SilkS)
@@
       (net 1 GND))
     (pad 1 thru_hole circle (at -3.5 -2.71 270) (size 1.9 1.9) (drill 0.92) (layers *.Cu *.Mask)
-      (net 1 GND))
-    (pad 2 thru_hole circle (at -1 -2.71 270) (size 1.9 1.9) (drill 0.92) (layers *.Cu *.Mask)
+      (net 8 "Net-(J2-Pad1)"))
+    (pad 2 thru_hole circle (at -1 -2.71 270) (size 1.8 1.8) (drill 0.92) (layers *.Cu *.Mask)
       (net 5 D-))
-    (pad 3 thru_hole circle (at 1 -2.71 270) (size 1.9 1.9) (drill 0.92) (layers *.Cu *.Mask)
+    (pad 3 thru_hole circle (at 1 -2.71 270) (size 1.8 1.8) (drill 0.92) (layers *.Cu *.Mask)
       (net 3 D+))
     (pad 4 thru_hole circle (at 3.5 -2.71 270) (size 1.9 1.9) (drill 0.92) (layers *.Cu *.Mask)
@@
   )
   (module Resistor_THT:R_Axial_DIN0207_L6.3mm_D2.5mm_P7.62mm_Horizontal (layer F.Cu)
-    (at 107.696 93.98 180)
+    (at 107.696 94.234 180)
     (descr "Resistor, Axial_DIN0207 series, Axial, Horizontal, pin pitch=7.62mm, 0.25W = 1/4W, length*diameter=6.3*2.5mm^2, http://cdn-reichelt.de/documents/datenblatt/B400/1_4W%23YAG.pdf")
     (tags "Resistor Axial_DIN0207 series Axial Horizontal pin pitch 7.62mm 0.25W = 1/4W length 6.3mm diameter 2.5mm")
@@
       (net 2 "Net-(D1-Pad1)"))
     (pad 2 thru_hole oval (at 7.62 0 180) (size 1.6 1.6) (drill 0.8) (layers *.Cu *.Mask)
-      (net 1 GND))
+      (net 8 "Net-(J2-Pad1)"))
     (model ${KISYS3DMOD}/Resistor_THT.3dshapes/R_Axial_DIN0207_L6.3mm_D2.5mm_P7.62mm_Horizontal.wrl
       (at (xyz 0 0 0))
@@
     )
     (pad 1 thru_hole rect (at 0 0) (size 1.9 1.9) (drill 0.9) (layers *.Cu *.Mask)
-      (net 1 GND))
+      (net 8 "Net-(J2-Pad1)"))
     (pad 2 thru_hole circle (at 2.5 0) (size 1.9 1.9) (drill 0.9) (layers *.Cu *.Mask)
       (net 4 "Net-(J1-Pad1)"))
@@
   (gr_line (start 134.874 121.92) (end 97.536 121.92) (layer Edge.Cuts) (width 0.05))
   (gr_line (start 134.874 90.932) (end 134.874 121.92) (layer Edge.Cuts) (width 0.05))
-  (segment (start 110.998 102.08) (end 110.914 102.164) (width 0.25) (layer F.Cu) (net 1))
-  (segment (start 110.858 102.108) (end 110.914 102.164) (width 0.25) (layer B.Cu) (net 1))
-  (segment (start 107.696 93.98) (end 111.506 93.98) (width 0.25) (layer F.Cu) (net 2))
+  (segment (start 107.696 94.234) (end 111.506 94.234) (width 0.25) (layer F.Cu) (net 2))
+  (segment (start 110.998 102.08) (end 110.914 102.164) (width 0.25) (layer F.Cu) (net 8))
+  (segment (start 110.858 102.108) (end 110.914 102.164) (width 0.25) (layer B.Cu) (net 8))
   (segment (start 114.538 106.664) (end 114.554 106.68) (width 1.7) (layer F.Cu) (net 3))
   (segment (start 110.914 106.664) (end 114.538 106.664) (width 1.7) (layer F.Cu) (net 3))
@@
   (segment (start 124.344 107.264) (end 125.222 107.264) (width 0.25) (layer F.Cu) (net 4))
   (segment (start 118.578 113.03) (end 124.344 107.264) (width 0.25) (layer F.Cu) (net 4))
-  (segment (start 126.689999 119.690001) (end 126.746 119.634) (width 3.4) (layer F.Cu) (net 5))
-  (segment (start 126.689999 119.690001) (end 126.689999 110.038001) (width 3.4) (layer F.Cu) (net 5))
   (segment (start 110.898 104.648) (end 110.914 104.664) (width 1.7) (layer F.Cu) (net 5))
   (segment (start 106.172 104.648) (end 110.898 104.648) (width 1.7) (layer F.Cu) (net 5))
@@
   (segment (start 103.124 104.648) (end 106.172 104.648) (width 3.4) (layer F.Cu) (net 5))
   (segment (start 103.124 116.078) (end 103.124 104.648) (width 3.4) (layer F.Cu) (net 5))
-  (segment (start 106.68 119.634) (end 103.124 116.078) (width 3.4) (layer F.Cu) (net 5))
-  (segment (start 109.869998 119.634) (end 106.68 119.634) (width 3.4) (layer F.Cu) (net 5))
-  (segment (start 109.925999 119.690001) (end 109.869998 119.634) (width 3.4) (layer F.Cu) (net 5))
-  (segment (start 126.689999 119.690001) (end 109.925999 119.690001) (width 3.4) (layer F.Cu) (net 5))
+  (segment (start 103.124 116.078) (end 103.378 116.078) (width 3.4) (layer F.Cu) (net 5))
+  (segment (start 103.378 116.078) (end 105.41 118.11) (width 3.4) (layer F.Cu) (net 5))
+  (segment (start 105.41 118.11) (end 126.746 118.11) (width 3.4) (layer F.Cu) (net 5))
+  (segment (start 126.746 110.094002) (end 126.689999 110.038001) (width 3.4) (layer F.Cu) (net 5))
+  (segment (start 126.746 118.11) (end 126.746 110.094002) (width 3.4) (layer F.Cu) (net 5))
+  (segment (start 110.914 102.164) (end 105.974 102.164) (width 0.25) (layer F.Cu) (net 8))
+  (segment (start 105.974 102.164) (end 100.076 96.266) (width 0.25) (layer F.Cu) (net 8))
+  (segment (start 116.078 107.328) (end 116.078 113.03) (width 0.25) (layer B.Cu) (net 8))
+  (segment (start 110.914 102.164) (end 116.078 107.328) (width 0.25) (layer B.Cu) (net 8))
+  (segment (start 100.076 94.234) (end 100.076 96.266) (width 0.25) (layer F.Cu) (net 8))
   (zone (net 1) (net_name GND) (layer B.Cu) (hatch edge 0.508)
     (connect_pads (clearance 0.508))
@@
     (polygon
       (pts
-        (xy 139.954 121.92) (xy 97.536 121.92) (xy 97.536 90.932) (xy 139.7 90.932)
+        (xy 134.874 121.92) (xy 97.536 121.92) (xy 97.536 90.932) (xy 134.874 90.932)
       )
     )

Commit message: So close, yet so far
Parts:
- moved D1 18.2 mm to (116.3, 112.3), turned to 180 degrees
- moved R1 16.9 mm to (118.9, 106.9), turned to 90 degrees
- moved S1 12.8 mm to (114.3, 100.3), turned to 270 degrees
- moved J2 5.11 mm to (103.6, 103.4)
- moved J1 0.92 mm to (126.1, 105.9)
Routing:
- net Net-(J2-Pad1): track 28.5 -> 13.1 mm
- net D-: track 55.5 -> 65.6 mm
- net Net-(J1-Pad1): track 9.91 -> 15.3 mm
- net D+: track 52.2 -> 57.1 mm
- net Net-(D1-Pad1): track 3.81 -> 5.33 mm
Other:
- board size 37.3 x 31 mm -> 42.7 x 38.3 mm
- rule trace_min: 0.152 -> 0.1524

Commit message: Made more changes to board and got closer but it still doesnt work
Parts:
- moved R1 0.91 mm to (118.8, 107.8)
Routing:
- net Net-(D1-Pad1): track 5.33 -> 4.39 mm
