File: PowerStripper.kicad_pcb (KiCad board)
At the start: 4 copper layers, 42.7 x 38.3 mm, 5 parts, among them J1 0548190519, J2 UE27AC54100

Commit message: trying to get it to export as 4 layers
Routing:
- added copper zone on L2, net GND
- added copper zone on L3, net GND
- removed copper zone on In1.Cu, net GND
- removed copper zone on In2.Cu, net GND
